Commit message: full description works with fakehardware (visu without bringup, uses joint state publisher gui)

File: src/diy_robotarm_wer24_description/urdf/common.urdf.xacro (robot description, xacro)
@@ -14,19 +14,25 @@
     <xacro:property name="shoulder_upper_limit" value="${sec_limits['shoulder']['max_position']}" scope="parent"/>
     <xacro:property name="shoulder_velocity_limit" value="${sec_limits['shoulder']['max_velocity']}" scope="parent"/>
+    <xacro:property name="shoulder_effort_limit" value="${sec_limits['shoulder']['max_effort']}" scope="parent"/>
     <xacro:property name="upper_arm_lower_limit" value="${sec_limits['upper_arm']['min_position']}" scope="parent"/>
     <xacro:property name="upper_arm_upper_limit" value="${sec_limits['upper_arm']['max_position']}" scope="parent"/>
     <xacro:property name="upper_arm_velocity_limit" value="${sec_limits['upper_arm']['max_velocity']}" scope="parent"/>
+    <xacro:property name="upper_arm_effort_limit" value="${sec_limits['upper_arm']['max_effort']}" scope="parent"/>
     <xacro:property name="forearm_lower_limit" value="${sec_limits['forearm']['min_position']}" scope="parent"/>
     <xacro:property name="forearm_upper_limit" value="${sec_limits['forearm']['max_position']}" scope="parent"/>
     <xacro:property name="forearm_velocity_limit" value="${sec_limits['forearm']['max_velocity']}" scope="parent"/>
+    <xacro:property name="forearm_effort_limit" value="${sec_limits['forearm']['max_effort']}" scope="parent"/>
     <xacro:property name="wrist_1_lower_limit" value="${sec_limits['wrist_1']['min_position']}" scope="parent"/>
     <xacro:property name="wrist_1_upper_limit" value="${sec_limits['wrist_1']['max_position']}" scope="parent"/>
     <xacro:property name="wrist_1_velocity_limit" value="${sec_limits['wrist_1']['max_velocity']}" scope="parent"/>
+    <xacro:property name="wrist_1_effort_limit" value="${sec_limits['wrist_1']['max_effort']}" scope="parent"/>
     <xacro:property name="wrist_2_lower_limit" value="${sec_limits['wrist_2']['min_position']}" scope="parent"/>
     <xacro:property name="wrist_2_upper_limit" value="${sec_limits['wrist_2']['max_position']}" scope="parent"/>
     <xacro:property name="wrist_2_velocity_limit" value="${sec_limits['wrist_2']['max_velocity']}" scope="parent"/>
+    <xacro:property name="wrist_2_effort_limit" value="${sec_limits['wrist_2']['max_effort']}" scope="parent"/>
     <xacro:property name="wrist_3_lower_limit" value="${sec_limits['wrist_3']['min_position']}" scope="parent"/>
     <xacro:property name="wrist_3_upper_limit" value="${sec_limits['wrist_3']['max_position']}" scope="parent"/>
     <xacro:property name="wrist_3_velocity_limit" value="${sec_limits['wrist_3']['max_velocity']}" scope="parent"/>
+    <xacro:property name="wrist_3_effort_limit" value="${sec_limits['wrist_3']['max_effort']}" scope="parent"/>
     <!-- kinematics -->
     <xacro:property name="shoulder_x" value="${sec_kinematics['shoulder']['x']}" scope="parent"/>

File: src/diy_robotarm_wer24_description/urdf/diy_robotarm_macro.urdf.xacro (robot description, xacro)
@@ -72,5 +72,5 @@
           keep_alive_count="${keep_alive_count}"
           />
-      </xacro:if>
+    </xacro:if>
 <!--#######################################################################################################################################-->
 <!--define the main kinematic chain with links and joints (using the config-files)-->
@@ -101,8 +101,8 @@
     <joint name="${tf_prefix}shoulder" type="revolute">
       <origin xyz="${shoulder_x} ${shoulder_y} ${shoulder_z}" rpy="${shoulder_roll} ${shoulder_pitch} ${shoulder_yaw}"/>
-      <parent link="base_link"/>
-      <child link="link_1"/>
-      <axis xyz="0.0 0.0 1.0"/>
-      <limit lower="${shoulder_lower_limit}" upper="${shoulder_upper_limit}" velocity="${shoulder_velocity_limit}"/>
+      <parent link="${tf_prefix}base_link"/>
+      <child link="${tf_prefix}link_1"/>
+      <axis xyz="0.0 0.0 1.0"/>
+      <limit lower="${shoulder_lower_limit}" upper="${shoulder_upper_limit}" velocity="${shoulder_velocity_limit}" effort="${shoulder_effort_limit}"/>
     </joint>
     <!-- Link1 = Shoulder -->
@@ -126,8 +126,8 @@
     <joint name="${tf_prefix}upper_arm" type="revolute">
       <origin xyz="${upper_arm_x} ${upper_arm_y} ${upper_arm_z}" rpy="${upper_arm_roll} ${upper_arm_pitch} ${upper_arm_yaw}"/>
-      <parent link="link_1"/>
-      <child link="link_2"/>
-      <axis xyz="0.0 0.0 1.0"/>
-      <limit lower="${upper_arm_lower_limit}" upper="${upper_arm_upper_limit}" velocity="${upper_arm_velocity_limit}"/>
+      <parent link="${tf_prefix}link_1"/>
+      <child link="${tf_prefix}link_2"/>
+      <axis xyz="0.0 0.0 1.0"/>
+      <limit lower="${upper_arm_lower_limit}" upper="${upper_arm_upper_limit}" velocity="${upper_arm_velocity_limit}" effort="${upper_arm_effort_limit}"/>
     </joint>
     <!-- Link2 = Upper_Arm -->
@@ -151,8 +151,8 @@
     <joint name="${tf_prefix}forearm" type="revolute">
       <origin xyz="${forearm_x} ${forearm_y} ${forearm_z}" rpy="${forearm_roll} ${forearm_pitch} ${forearm_yaw}"/>
-      <parent link="link_2"/>
-      <child link="link_3"/>
-      <axis xyz="0.0 0.0 1.0"/>
-      <limit lower="${forearm_lower_limit}" upper="${forearm_upper_limit}" velocity="${forearm_velocity_limit}"/>
+      <parent link="${tf_prefix}link_2"/>
+      <child link="${tf_prefix}link_3"/>
+      <axis xyz="0.0 0.0 1.0"/>
+      <limit lower="${forearm_lower_limit}" upper="${forearm_upper_limit}" velocity="${forearm_velocity_limit}" effort="${forearm_effort_limit}"/>
     </joint>
     <!-- Link3 = Forearm -->
@@ -176,8 +176,8 @@
     <joint name="${tf_prefix}wrist_1" type="revolute">
       <origin xyz="${wrist_1_x} ${wrist_1_y} ${wrist_1_z}" rpy="${wrist_1_roll} ${wrist_1_pitch} ${wrist_1_yaw}"/>
-      <parent link="link_3"/>
-      <child link="link_4"/>
-      <axis xyz="0.0 0.0 1.0"/>
-      <limit lower="${wrist_1_lower_limit}" upper="${wrist_1_upper_limit}" velocity="${wrist_1_velocity_limit}"/>
+      <parent link="${tf_prefix}link_3"/>
+      <child link="${tf_prefix}link_4"/>
+      <axis xyz="0.0 0.0 1.0"/>
+      <limit lower="${wrist_1_lower_limit}" upper="${wrist_1_upper_limit}" velocity="${wrist_1_velocity_limit}" effort="${wrist_1_effort_limit}"/>
     </joint>
     <!-- Link4 = Wrist 1 -->
@@ -201,8 +201,8 @@
     <joint name="${tf_prefix}wrist_2" type="revolute">
       <origin xyz="${wrist_2_x} ${wrist_2_y} ${wrist_2_z}" rpy="${wrist_2_roll} ${wrist_2_pitch} ${wrist_2_yaw}"/>
-      <parent link="link_4"/>
-      <child link="link_5"/>
-      <axis xyz="0.0 0.0 1.0"/>
-      <limit lower="${wrist_2_lower_limit}" upper="${wrist_2_upper_limit}" velocity="${wrist_2_velocity_limit}"/>
+      <parent link="${tf_prefix}link_4"/>
+      <child link="${tf_prefix}link_5"/>
+      <axis xyz="0.0 0.0 1.0"/>
+      <limit lower="${wrist_2_lower_limit}" upper="${wrist_2_upper_limit}" velocity="${wrist_2_velocity_limit}" effort="${wrist_2_effort_limit}"/>
     </joint>
     <!-- Link5 = Wrist 2 -->
@@ -226,8 +226,8 @@
     <joint name="${tf_prefix}wrist_3" type="revolute">
       <origin xyz="${wrist_3_x} ${wrist_3_y} ${wrist_3_z}" rpy="${wrist_3_roll} ${wrist_3_pitch} ${wrist_3_yaw}"/>
-      <parent link="link_5"/>
-      <child link="link_6"/>
-      <axis xyz="0.0 0.0 1.0"/>
-      <limit lower="${wrist_3_lower_limit}" upper="${wrist_3_upper_limit}" velocity="${wrist_3_velocity_limit}"/>
+      <parent link="${tf_prefix}link_5"/>
+      <child link="${tf_prefix}link_6"/>
+      <axis xyz="0.0 0.0 1.0"/>
+      <limit lower="${wrist_3_lower_limit}" upper="${wrist_3_upper_limit}" velocity="${wrist_3_velocity_limit}" effort="${wrist_3_effort_limit}"/>
     </joint>
     <!-- Link6 = Flange -->
