Commit message: delete force abs path in common.urdf

File: urdf/common.urdf.xacro (robot description, xacro)
@@ -2,6 +2,5 @@
 <!-- this file includes helper macros to unpack configs frim .yaml files and pass them into properties, callable in the outer macros-->
 <robot xmlns:xacro="http://wiki.ros.org/xacro">
-  <xacro:macro name="read_model_data" params="joint_limits_parameters_file kinematics_parameters_file  force_abs_paths">
-    <xacro:property name="force_abs_paths" value="${force_abs_paths}" scope="parent"/>
+  <xacro:macro name="read_model_data" params="joint_limits_parameters_file kinematics_parameters_file">
     <!-- Read .yaml files from disk, load content into properties -->
     <xacro:property name="config_joint_limit_parameters" value="${xacro.load_yaml(joint_limits_parameters_file)}"/>
