Commit message: implemented tf_prefix for materials to avoid name collisions

File: urdf/diy_robotarm_macro.urdf.xacro (robot description, xacro)
@@ -76,4 +76,5 @@
 <!--define the main kinematic chain with links and joints (using the config-files)-->
 <!--#######################################################################################################################################-->
+    <xacro:materials tf_prefix="${tf_prefix}"/>
     <!-- Achse fix Base to parent passed in the main_urdf.xacro-->
     <joint name="${tf_prefix}robotarm_to_parent" type="fixed">

File: urdf/materials.urdf.xacro (robot description, xacro)
@@ -4,31 +4,33 @@
 https://github.com/ros-simulation/gazebo_ros_demos/blob/kinetic-devel/rrbot_description/urdf/materials.xacro
 -->
-<robot>
-  <material name="black">
-    <color rgba="0.0 0.0 0.0 1.0"/>
-  </material>
-  <material name="blue">
-    <color rgba="0.0 0.0 0.8 1.0"/>
-  </material>
-  <material name="green">
-    <color rgba="0.0 0.8 0.0 1.0"/>
-  </material>
-  <material name="yellow">
-    <color rgba="1.0 1.0 0.0 1.0"/>
-  </material>
-  <material name="grey">
-    <color rgba="0.6 0.6 0.6 1.0"/>
-  </material>
-  <material name="orange">
-    <color rgba="${255/255} ${108/255} ${10/255} 1.0"/>
-  </material>
-  <material name="brown">
-    <color rgba="${222/255} ${207/255} ${195/255} 1.0"/>
-  </material>
-  <material name="red">
-    <color rgba="0.8 0.0 0.0 1.0"/>
-  </material>
-  <material name="white">
-    <color rgba="1.0 1.0 1.0 1.0"/>
-  </material>
+<robot xmlns:xacro="http://wiki.ros.org/xacro">
+  <xacro:macro name="materials" params="tf_prefix">
+    <material name="${tf_prefix}black">
+      <color rgba="0.0 0.0 0.0 1.0"/>
+    </material>
+    <material name="${tf_prefix}blue">
+      <color rgba="0.0 0.0 0.8 1.0"/>
+    </material>
+    <material name="${tf_prefix}green">
+      <color rgba="0.0 0.8 0.0 1.0"/>
+    </material>
+    <material name="${tf_prefix}yellow">
+      <color rgba="1.0 1.0 0.0 1.0"/>
+    </material>
+    <material name="${tf_prefix}grey">
+      <color rgba="0.6 0.6 0.6 1.0"/>
+    </material>
+    <material name="${tf_prefix}orange">
+      <color rgba="${255/255} ${108/255} ${10/255} 1.0"/>
+    </material>
+    <material name="${tf_prefix}brown">
+      <color rgba="${222/255} ${207/255} ${195/255} 1.0"/>
+    </material>
+    <material name="${tf_prefix}red">
+      <color rgba="0.8 0.0 0.0 1.0"/>
+    </material>
+    <material name="${tf_prefix}white">
+      <color rgba="1.0 1.0 1.0 1.0"/>
+    </material>
+  </xacro:macro>
 </robot>

Commit message: add tf_prefix to material troubleshooting

File: urdf/diy_robotarm_macro.urdf.xacro (robot description, xacro)
@@ -114,5 +114,5 @@
           <mesh filename="package://diy_robotarm_wer24_description/meshes/visual/link_1.stl" scale="0.001 0.001 0.001"/>
         </geometry>
-        <material name="grey"/>
+        <material name="${tf_prefix}grey"/>
       </visual>
        <!-- <collision>
@@ -139,5 +139,5 @@
           <mesh filename="package://diy_robotarm_wer24_description/meshes/visual/link_2.stl" scale="0.001 0.001 0.001"/>
         </geometry>
-        <material name="grey"/>
+        <material name="${tf_prefix}grey"/>
       </visual>
       <!-- <collision>
@@ -164,5 +164,5 @@
           <mesh filename="package://diy_robotarm_wer24_description/meshes/visual/link_3.stl" scale="0.001 0.001 0.001"/>
         </geometry>
-        <material name="grey"/>
+        <material name="${tf_prefix}grey"/>
       </visual>
       <!-- <collision>
@@ -189,5 +189,5 @@
           <mesh filename="package://diy_robotarm_wer24_description/meshes/visual/link_4.stl" scale="0.001 0.001 0.001"/>
         </geometry>
-        <material name="grey"/>
+        <material name="${tf_prefix}grey"/>
       </visual>
       <!-- <collision>
@@ -214,5 +214,5 @@
           <mesh filename="package://diy_robotarm_wer24_description/meshes/visual/link_5.stl" scale="0.001 0.001 0.001"/>
         </geometry>
-        <material name="grey"/>
+        <material name="${tf_prefix}grey"/>
       </visual>
       <!-- <collision>
@@ -239,5 +239,5 @@
           <mesh filename="package://diy_robotarm_wer24_description/meshes/visual/link_6.stl" scale="0.001 0.001 0.001"/>
         </geometry>
-        <material name="grey"/>
+        <material name="${tf_prefix}grey"/>
       </visual>
       <!-- <collision>

Commit message: materials_troubleshooting

File: urdf/diy_robotarm_macro.urdf.xacro (robot description, xacro)
@@ -89,5 +89,5 @@
           <mesh filename="package://diy_robotarm_wer24_description/meshes/visual/base.stl" scale="0.001 0.001 0.001"/>
         </geometry>
-        <material name="grey"/>
+        <material name="${tf_prefix}grey"/>
       </visual>
       <!-- <collision>

Commit message: add collision properties to macro.urdf

File: urdf/diy_robotarm_macro.urdf.xacro (robot description, xacro)
@@ -34,5 +34,4 @@
   <!--include ros2 control and create an instance if param generate_ros2_control_tag == true and pass necessary params-->
   <!--#######################################################################################################################################-->
-  <!--still to modify delete not necessary params-->
     <xacro:if value="${generate_ros2_control_tag}">
         <!-- ros2 control include -->
@@ -67,11 +66,11 @@
         <material name="${tf_prefix}grey"/>
       </visual>
-      <!-- <collision>
+      <collision>
         <origin xyz="0 0 0 rpy = 0 0 0"/>
         <geometry>
           <mesh filename="package://diy_robotarm_wer24_description/meshes/collision/base.stl" scale="0.001 0.001 0.001"/>
         </geometry>
-        <material name="red"/>
-      </collision> -->
+        <material name="${tf_prefix}red"/>
+      </collision>
     </link>
     <!-- Achse 1 (Base = World)-->
@@ -92,11 +91,11 @@
         <material name="${tf_prefix}grey"/>
       </visual>
-       <!-- <collision>
+      <collision>
         <origin xyz="0 0 0 rpy = 0 0 0"/>
         <geometry>
           <mesh filename="package://diy_robotarm_wer24_description/meshes/collision/link_1.stl" scale="0.001 0.001 0.001"/>
         </geometry>
-        <material name="red"/>
-      </collision> -->
+        <material name="${tf_prefix}red"/>
+      </collision>
     </link>
     <!-- Achse 2 -->
@@ -117,11 +116,11 @@
         <material name="${tf_prefix}grey"/>
       </visual>
-      <!-- <collision>
+      <collision>
         <origin xyz="0 0 0 rpy = 0 0 0"/>
         <geometry>
           <mesh filename="package://diy_robotarm_wer24_description/meshes/collision/link_2.stl" scale="0.001 0.001 0.001"/>
         </geometry>
-        <material name="red"/>
-      </collision> -->
+        <material name="${tf_prefix}red"/>
+      </collision>
     </link>
     <!-- Achse 3 -->
@@ -142,11 +141,11 @@
         <material name="${tf_prefix}grey"/>
       </visual>
-      <!-- <collision>
+      <collision>
         <origin xyz="0 0 0 rpy = 0 0 0"/>
         <geometry>
           <mesh filename="package://diy_robotarm_wer24_description/meshes/collision/link_3.stl" scale="0.001 0.001 0.001"/>
         </geometry>
-        <material name="red"/>
-      </collision> -->
+        <material name="${tf_prefix}red"/>
+      </collision>
     </link>
     <!-- Achse 4 -->
@@ -167,11 +166,11 @@
         <material name="${tf_prefix}grey"/>
       </visual>
-      <!-- <collision>
+      <collision>
         <origin xyz="0 0 0 rpy = 0 0 0"/>
         <geometry>
           <mesh filename="package://diy_robotarm_wer24_description/meshes/collision/link_4.stl" scale="0.001 0.001 0.001"/>
         </geometry>
-        <material name="red"/>
-      </collision> -->
+        <material name="${tf_prefix}red"/>
+      </collision>
     </link>
     <!-- Achse 5 -->
@@ -192,11 +191,11 @@
         <material name="${tf_prefix}grey"/>
       </visual>
-      <!-- <collision>
+      <collision>
         <origin xyz="0 0 0 rpy = 0 0 0"/>
         <geometry>
           <mesh filename="package://diy_robotarm_wer24_description/meshes/collision/link_5.stl" scale="0.001 0.001 0.001"/>
         </geometry>
-        <material name="red"/>
-      </collision> -->
+        <material name="${tf_prefix}red"/>
+      </collision>
     </link>
     <!-- Achse 6 -->
@@ -217,11 +216,11 @@
         <material name="${tf_prefix}grey"/>
       </visual>
-      <!-- <collision>
+      <collision>
         <origin xyz="0 0 0 rpy = 0 0 0"/>
         <geometry>
           <mesh filename="package://diy_robotarm_wer24_description/meshes/collision/link_6.stl" scale="0.001 0.001 0.001"/>
         </geometry>
-        <material name="red"/>
-      </collision> -->
+        <material name="${tf_prefix}red"/>
+      </collision>
     </link>
   </xacro:macro>

Commit message: deleted rpy for masecone, wrong sytax

File: urdf/diy_robotarm_macro.urdf.xacro (robot description, xacro)
@@ -67,5 +67,5 @@
       </visual>
       <collision>
-        <origin xyz="0 0 0 rpy = 0 0 0"/>
+        <origin xyz="0 0 0"/>
         <geometry>
           <mesh filename="package://diy_robotarm_wer24_description/meshes/collision/base.stl" scale="0.001 0.001 0.001"/>

Commit message: rpy error link 1-6 solved

File: urdf/diy_robotarm_macro.urdf.xacro (robot description, xacro)
@@ -91,5 +91,5 @@
       </visual>
       <collision>
-        <origin xyz="0 0 0 rpy = 0 0 0"/>
+        <origin xyz="0 0 0" rpy = "0 0 0"/>
         <geometry>
           <mesh filename="package://diy_robotarm_wer24_description/meshes/collision/link_1.stl" scale="0.001 0.001 0.001"/>
@@ -116,5 +116,5 @@
       </visual>
       <collision>
-        <origin xyz="0 0 0 rpy = 0 0 0"/>
+        <origin xyz="0 0 0" rpy = "0 0 0"/>
         <geometry>
           <mesh filename="package://diy_robotarm_wer24_description/meshes/collision/link_2.stl" scale="0.001 0.001 0.001"/>
@@ -141,5 +141,5 @@
       </visual>
       <collision>
-        <origin xyz="0 0 0 rpy = 0 0 0"/>
+        <origin xyz="0 0 0" rpy = "0 0 0"/>
         <geometry>
           <mesh filename="package://diy_robotarm_wer24_description/meshes/collision/link_3.stl" scale="0.001 0.001 0.001"/>
@@ -166,5 +166,5 @@
       </visual>
       <collision>
-        <origin xyz="0 0 0 rpy = 0 0 0"/>
+        <origin xyz="0 0 0" rpy = "0 0 0"/>
         <geometry>
           <mesh filename="package://diy_robotarm_wer24_description/meshes/collision/link_4.stl" scale="0.001 0.001 0.001"/>
@@ -191,5 +191,5 @@
       </visual>
       <collision>
-        <origin xyz="0 0 0 rpy = 0 0 0"/>
+        <origin xyz="0 0 0" rpy = "0 0 0"/>
         <geometry>
           <mesh filename="package://diy_robotarm_wer24_description/meshes/collision/link_5.stl" scale="0.001 0.001 0.001"/>
@@ -216,5 +216,5 @@
       </visual>
       <collision>
-        <origin xyz="0 0 0 rpy = 0 0 0"/>
+        <origin xyz="0 0 0" rpy = "0 0 0"/>
         <geometry>
           <mesh filename="package://diy_robotarm_wer24_description/meshes/collision/link_6.stl" scale="0.001 0.001 0.001"/>
